File: PCB/m0module.kicad_pcb (KiCad board)
At the start: 2 copper layers, 18 x 22 mm, 24 parts, among them J2 TEST_1P, J4 TEST_1P, SW4 SW_PUSH, U1 MIC5353-3.3YMT-TR, U2 SAMD21G18, U4 SAMD21_MOD, Y1 Crystal_Small

Commit message: Boards ordered wth gerbs
Other:
- board text added: "RX"
- board text added: "TX"
- board text added: "bridge_mod v01p"
Changed lines of the file:
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@@
-(kicad_pcb (version 4) (host pcbnew 4.0.7)
+(kicad_pcb (version 4) (host pcbnew 4.0.4-stable)
   (general
     (links 110)
@@
     (area 61.42 50.05 138.435747 118.750001)
     (thickness 1.6)
-    (drawings 4)
+    (drawings 9)
     (tracks 569)
     (zones 0)
@@
     (visible_elements 7FFFEE7F)
     (pcbplotparams
-      (layerselection 0x010f0_80000001)
+      (layerselection 0x010fc_80000001)
       (usegerberextensions false)
       (excludeedgelayer true)
@@
     )
   )
+  (dimension 22.000227 (width 0.3) (layer Cmts.User)
+    (gr_text "22.000 mm" (at 125.173729 88.917255 270.2604336) (layer Cmts.User)
+      (effects (font (size 1.5 1.5) (thickness 0.3)))
+    )
+    (feature1 (pts (xy 117.92 77.95) (xy 126.473715 77.911119)))
+    (feature2 (pts (xy 118.02 99.95) (xy 126.573715 99.911119)))
+    (crossbar (pts (xy 123.873743 99.923392) (xy 123.773743 77.923392)))
+    (arrow1a (pts (xy 123.773743 77.923392) (xy 124.365278 79.047219)))
+    (arrow1b (pts (xy 123.773743 77.923392) (xy 123.192449 79.05255)))
+    (arrow2a (pts (xy 123.873743 99.923392) (xy 124.455037 98.794234)))
+    (arrow2b (pts (xy 123.873743 99.923392) (xy 123.282208 98.799565)))
+  )
+  (dimension 18.000069 (width 0.3) (layer Cmts.User)
+    (gr_text "18.000 mm" (at 109.041486 107.660084 0.1591545337) (layer Cmts.User)
+      (effects (font (size 1.5 1.5) (thickness 0.3)))
+    )
+    (feature1 (pts (xy 118.02 99.9) (xy 118.045236 108.985079)))
+    (feature2 (pts (xy 100.02 99.95) (xy 100.045236 109.035079)))
+    (crossbar (pts (xy 100.037736 106.335089) (xy 118.037736 106.285089)))
+    (arrow1a (pts (xy 118.037736 106.285089) (xy 116.912866 106.874637)))
+    (arrow1b (pts (xy 118.037736 106.285089) (xy 116.909608 105.7018)))
+    (arrow2a (pts (xy 100.037736 106.335089) (xy 101.165864 106.918378)))
+    (arrow2b (pts (xy 100.037736 106.335089) (xy 101.162606 105.745541)))
+  )
+  (gr_text "bridge_mod v01p\n" (at 102.07 85.95 90) (layer B.Paste)
+    (effects (font (size 1 1) (thickness 0.25)) (justify mirror))
+  )
+  (gr_text "TX\n" (at 102.77 96.45) (layer F.SilkS)
+    (effects (font (size 1 1) (thickness 0.25)))
+  )
+  (gr_text RX (at 114.77 96.15) (layer F.SilkS)
+    (effects (font (size 1 1) (thickness 0.25)))
+  )
   (gr_line (start 118 100) (end 100 100) (layer Edge.Cuts) (width 0.1))
