File: demo_boards/lipo_charge_mod/lipo_charge_mod.kicad_pcb (KiCad board)
At the start: 2 copper layers, 18 x 7 mm, 9 parts, among them J1 GS3, J2 Conn_01x06, U5 MCP73831T

Commit message: added demo boards
Other:
- board text added: "LIPO_CHARGE_MOD"
Changed lines of the file:
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@@
-(kicad_pcb (version 4) (host pcbnew 4.0.7)
+(kicad_pcb (version 4) (host pcbnew 4.0.4-stable)
   (general
     (links 25)
-    (no_connects 11)
-    (area 92.219999 86.109999 110.320001 93.210001)
+    (no_connects 0)
+    (area 61.42 50.05 138.435747 118.750001)
     (thickness 1.6)
-    (drawings 4)
+    (drawings 7)
     (tracks 35)
     (zones 0)
@@
   )
   (setup
-    (last_trace_width 1)
+    (last_trace_width 0.2)
     (user_trace_width 0.2)
     (user_trace_width 0.4)
@@
     )
   )
+  (dimension 7 (width 0.3) (layer Cmts.User)
+    (gr_text "7.000 mm" (at 113.62 89.66 90) (layer Cmts.User)
+      (effects (font (size 1.5 1.5) (thickness 0.3)))
+    )
+    (feature1 (pts (xy 108.27 86.16) (xy 114.97 86.16)))
+    (feature2 (pts (xy 108.27 93.16) (xy 114.97 93.16)))
+    (crossbar (pts (xy 112.27 93.16) (xy 112.27 86.16)))
+    (arrow1a (pts (xy 112.27 86.16) (xy 112.856421 87.286504)))
+    (arrow1b (pts (xy 112.27 86.16) (xy 111.683579 87.286504)))
+    (arrow2a (pts (xy 112.27 93.16) (xy 112.856421 92.033496)))
+    (arrow2b (pts (xy 112.27 93.16) (xy 111.683579 92.033496)))
+  )
+  (dimension 18 (width 0.3) (layer Cmts.User)
+    (gr_text "18.000 mm" (at 101.27 97.51) (layer Cmts.User)
+      (effects (font (size 1.5 1.5) (thickness 0.3)))
+    )
+    (feature1 (pts (xy 110.27 92.16) (xy 110.27 98.86)))
+    (feature2 (pts (xy 92.27 92.16) (xy 92.27 98.86)))
+    (crossbar (pts (xy 92.27 96.16) (xy 110.27 96.16)))
+    (arrow1a (pts (xy 110.27 96.16) (xy 109.143496 96.746421)))
+    (arrow1b (pts (xy 110.27 96.16) (xy 109.143496 95.573579)))
+    (arrow2a (pts (xy 92.27 96.16) (xy 93.396504 96.746421)))
+    (arrow2b (pts (xy 92.27 96.16) (xy 93.396504 95.573579)))
+  )
+  (gr_text LIPO_CHARGE_MOD (at 101.27 92.16) (layer B.SilkS)
+    (effects (font (size 1 1) (thickness 0.25)) (justify mirror))
+  )
   (gr_line (start 110.27 93.16) (end 92.27 93.16) (layer Edge.Cuts) (width 0.1))
