File: demo_boards/Cherry MX Board/hcc_cherry.kicad_pcb (KiCad board)
At the start: 2 copper layers, 77 x 77 mm, 23 parts, among them J1 USB_B, J10 GS3, J2 SW1, J3 SW2, J4 SW3, J5 SW4, J6 SW5, J7 SW6, J8 SW7, J9 SW8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

Commit message: Fixed USB Ground
Parts:
- J1: value USB_B -> USB_OTG
Connections:
- J1 pad 4: GND -> Net-(J1-Pad4)
- J1 pad 5: Net-(J1-Pad5) -> GND
- J1 pad 6: (no net) -> Net-(J1-Pad6)

Commit message: updated hcc mod and modzilla board gerbs
Connections:
- C1 pad 1: Net-(C1-Pad1) -> +3V3
- C2 pad 1: Net-(C1-Pad1) -> +3V3
- J10 pad 2: Net-(C1-Pad1) -> +3V3
- U1 pad 1: Net-(C1-Pad1) -> +3V3
- U2 pad 1: Net-(C1-Pad1) -> +3V3
- U3 pad 1: Net-(C1-Pad1) -> +3V3
- U5 pad 1: Net-(C1-Pad1) -> +3V3
- U6 pad 1: Net-(C1-Pad1) -> +3V3
- U7 pad 1: Net-(C1-Pad1) -> +3V3
- U8 pad 1: Net-(C1-Pad1) -> +3V3
- U9 pad 1: Net-(C1-Pad1) -> +3V3
Routing:
- net +3V3: track 39.1 -> 200.4 mm, vias 0 -> 2
- net Net-(C1-Pad1): track 160.2 -> 0.00 mm, vias 2 -> 0

Commit message: connected 3V3 to LEDs without needing jumper
Other:
- board text added: "Cherry MX Demo Board for the HCC Module IdleHandsDev.com youtube.com/SeanHodginsFilms"
Changed lines of the file:
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@@
     (links 67)
     (no_connects 6)
-    (area 161.569999 102.199999 238.670001 179.300001)
+    (area 137.442 84.086 263.680001 191.272001)
     (thickness 1.6)
-    (drawings 28)
+    (drawings 29)
     (tracks 200)
     (zones 0)
@@
       (xy 6.670737 -4.683673) (xy 6.739949 -4.686874) (xy 6.788154 -4.672533)) (layer F.SilkS) (width 0.01))
   )
+  (gr_text "Cherry MX Demo Board for the HCC Module\nIdleHandsDev.com\nyoutube.com/SeanHodginsFilms" (at 226.12 173.95) (layer B.SilkS)
+    (effects (font (size 1.5 1.5) (thickness 0.3)) (justify left mirror))
+  )
   (dimension 77.5 (width 0.3) (layer Cmts.User)

Commit message: cleaned up libs, removed libs from project files, removed unused footprints
Other:
- outline, holes or cut-outs redrawn
Changed lines of the file:
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@@
   (general
     (links 67)
-    (no_connects 6)
+    (no_connects 5)
     (area 137.442 84.086 263.680001 191.272001)
     (thickness 1.6)
-    (drawings 29)
+    (drawings 21)
     (tracks 200)
     (zones 0)
@@
   (gr_circle (center 164.62 176.286) (end 166.12 176.286) (layer Dwgs.User) (width 0.1))
   (gr_arc (start 164.62 136.551981) (end 163.843543 133.654203) (angle -75) (layer Edge.Cuts) (width 0.1))
-  (gr_circle (center 171.62 167.25) (end 172.62 167.25) (layer Edge.Cuts) (width 0.1))
   (gr_arc (start 210.62 118.014661) (end 211.396457 120.912438) (angle -75) (layer Edge.Cuts) (width 0.1))
   (gr_line (start 211.396457 120.912438) (end 163.843543 133.654203) (layer Edge.Cuts) (width 0.1))
@@
   (gr_arc (start 216.62 105.25) (end 216.62 102.25) (angle -90) (layer Edge.Cuts) (width 0.1))
   (gr_line (start 161.62 136.551981) (end 161.62 176.25) (layer Edge.Cuts) (width 0.1))
-  (gr_circle (center 228.62 167.25) (end 229.62 167.25) (layer Edge.Cuts) (width 0.1))
-  (gr_circle (center 209.62 167.25) (end 210.62 167.25) (layer Edge.Cuts) (width 0.1))
   (gr_circle (center 216.62 105.25) (end 217.62 105.25) (layer Edge.Cuts) (width 0.1))
   (gr_circle (center 235.62 105.25) (end 236.62 105.25) (layer Edge.Cuts) (width 0.1))
@@
   (gr_arc (start 235.62 105.25) (end 238.62 105.25) (angle -90) (layer Edge.Cuts) (width 0.1))
   (gr_line (start 235.62 102.25) (end 216.62 102.25) (layer Edge.Cuts) (width 0.1))
-  (gr_circle (center 228.62 148.25) (end 229.62 148.25) (layer Edge.Cuts) (width 0.1))
-  (gr_circle (center 190.62 148.25) (end 191.62 148.25) (layer Edge.Cuts) (width 0.1))
-  (gr_circle (center 171.62 148.25) (end 172.62 148.25) (layer Edge.Cuts) (width 0.1))
-  (gr_circle (center 190.62 167.25) (end 191.62 167.25) (layer Edge.Cuts) (width 0.1))
-  (gr_circle (center 209.62 148.25) (end 210.62 148.25) (layer Edge.Cuts) (width 0.1))
   (segment (start 235.12 131.45) (end 237.142 131.45) (width 0.4) (layer F.Cu) (net 1))
   (segment (start 237.142 131.45) (end 237.264 131.328) (width 0.4) (layer F.Cu) (net 1))
